File: Aquarium_LED_Dimmer.kicad_pcb (KiCad board)
At the start: 2 copper layers, 69.2 x 25 mm, 33 parts, among them Q1 DGM3418L-7, U1 NE555D, U2 LM2674M-12

Commit message: Add files via upload
Parts:
- D5: renamed from PWR; value LED_Green -> PWR
- R4, R7: value ?k -> 1.8k
- R5: value ?k -> 1k
- moved RV1 0.74 mm to (174.3, 94.5)
Routing:
- net Net-(D4-Pad2): track 12.5 -> 11.7 mm
- net Net-(C5-Pad1): track 22.0 -> 22.7 mm
- net Net-(D3-Pad1): track 14.8 -> 14.2 mm
